Commit message: Added skybox, changed floor, changed camera resolution

File: gym_pybullet_drones/assets/envmap/plane.urdf (robot description, URDF)
Before this commit: robot plane, 1 links, 0 joints
Links:
- link planeLink: geometry collision box size=300 300 10; visual mesh filename=ground_texture/aerial_grass_rock_2k.obj scale=1 1 1

File: gym_pybullet_drones/assets/envmap/sky.urdf (robot description, URDF)
Before this commit: robot sky, 1 links, 0 joints
Links:
- removed link skyLink
- added link skyLink1, mass .0; visual mesh filename=skymap_texture/sky_1.obj scale=1 1 1
- added link skyLink2, mass .0; visual mesh filename=skymap_texture/sky_2.obj scale=1 1 1
- added link skyLink3, mass .0; visual mesh filename=skymap_texture/sky_3.obj scale=1 1 1
- added link skyLink4, mass .0; visual mesh filename=skymap_texture/sky_4.obj scale=1 1 1
Joints:
- added joint skyLink1_to_skyLink2: type fixed, parent skyLink1, child skyLink2, origin xyz=0 0 0 rpy=0 0 0
- added joint skyLink2_to_skyLink3: type fixed, parent skyLink2, child skyLink3, origin xyz=0 0 0 rpy=0 0 0
- added joint skyLink3_to_skyLink4: type fixed, parent skyLink3, child skyLink4, origin xyz=0 0 0 rpy=0 0 0
